Commit message: change to flexiv robot

File: urdf2model/models/mabimobile/mabi_mobile.urdf (robot description, URDF)
Before this commit: robot mabi_mobile, 40 links, 39 joints
Links:
- removed link ARM
- removed link BASE_ADAPTER_1
- removed link BASE_FORCETORQUESENSOR
- removed link BASE_IMU
- removed link EE_FORCETORQUESENSOR
- removed link EE_IMU
- removed link ELBOW
- removed link ENDEFFECTOR
- removed link FOREARM
- removed link FT_FLANGE
- removed link GRIPPER_BASE
- removed link GRIPPER_left_coupler
- removed link GRIPPER_left_driver
- removed link GRIPPER_left_follower
- removed link GRIPPER_left_pad
- removed link GRIPPER_left_spring_link
- removed link GRIPPER_right_coupler
- removed link GRIPPER_right_driver
- removed link GRIPPER_right_follower
- removed link GRIPPER_right_pad
- removed link GRIPPER_right_spring_link
- removed link SHOULDER
- removed link WRIST_1
- removed link WRIST_2
- removed link arm_mount
- removed link base_footprint
- removed link camera_mount
- removed link camera_vr_orientation
- removed link imu_link
- removed link realsense_odom_input_frame
- removed link robotiq_coupler
- added link base_acc
- added link base_gps
- added link base_gyro
- added link base_inertial
- added link link1
- added link link2
- added link link3
- added link link4
- added link link5
- added link link6
- added link link7
- link L_WHEEL: mass 10.9 -> None; geometry collision cylinder length=0.06 radius=0.15; visual cylinder length=0.06 radius=0.15
- link R_WHEEL: mass 10.9 -> None; geometry collision cylinder length=0.06 radius=0.15; visual cylinder length=0.06 radius=0.15
- link arm_base: mass 0.0001 -> None
- link base_link: geometry collision box size=0.02 0.7 0.289; collision box size=0.02 0.7 0.289
- link base_link_inertia: mass 60 -> None
- link cw_fl_link: mass 3.0 -> None; geometry collision cylinder length=0.04 radius=0.05; visual cylinder length=0.04 radius=0.05
- link cw_fr_link: mass 3.0 -> None; geometry collision cylinder length=0.04 radius=0.05; visual cylinder length=0.04 radius=0.05
- link cw_hl_link: mass 3.0 -> None; geometry collision cylinder length=0.04 radius=0.05; visual cylinder length=0.04 radius=0.05
- link cw_hr_link: mass 3.0 -> None; geometry collision cylinder length=0.04 radius=0.05; visual cylinder length=0.04 radius=0.05
Joints:
- removed joint BASE_ADAPTER_1_JOINT
- removed joint BASE_FORCETORQUESENSOR_FRAME
- removed joint BASE_FORCETORQUESENSOR_JOINT
- removed joint BASE_IMU_JOINT
- removed joint EE_FORCETORQUESENSOR_FRAME
- removed joint EE_FORCETORQUESENSOR_JOINT
- removed joint EE_IMU_JOINT
- removed joint EL_FLE
- removed joint EL_ROT
- removed joint GRIPPER_BASE_ENDEFFECTOR_JOINT
- removed joint GRIPPER_JOINT
- removed joint GRIPPER_left_coupler_joint
- removed joint GRIPPER_left_driver_joint
- removed joint GRIPPER_left_follower_joint
- removed joint GRIPPER_left_pad_joint
- removed joint GRIPPER_left_spring_link_joint
- removed joint GRIPPER_right_coupler_joint
- removed joint GRIPPER_right_follower_joint
- removed joint GRIPPER_right_pad_joint
- removed joint GRIPPER_right_spring_link_joint
- removed joint J_L_WHEEL
- removed joint J_R_WHEEL
- removed joint SH_FLE
- removed joint SH_ROT
- removed joint WR_FLE
- removed joint WR_ROT
- removed joint base_footprint_joint
- removed joint base_to_arm_base
- removed joint base_to_camera_mount
- removed joint base_to_realsense_odom_input_frame
- removed joint camera_ros_to_vr_convention
- removed joint cw_fl
- removed joint cw_fr
- removed joint cw_hl
- removed joint cw_hr
- removed joint imu_joint
- removed joint inertial_joint
- removed joint robotiq_coupler_GRIPPER_BASE_joint
- removed joint robotiq_coupler_coupler_joint
- added joint L_WHEEL: type fixed, parent base_link, child L_WHEEL, origin xyz=0 0.29 0.1 rpy=0 0 0, axis 0 1 0, limit effort=50 velocity=10
- added joint R_WHEEL: type fixed, parent base_link, child R_WHEEL, origin xyz=0 -0.29 0.1 rpy=0 0 0, axis 0 1 0, limit effort=50 velocity=10
- added joint base_link_arm_base_joint: type fixed, parent base_link, child arm_base, origin xyz=0 0 0.309 rpy=0 0 0
- added joint base_link_base_acc_joint: type fixed, parent base_link, child base_acc, origin xyz=0 0 0 rpy=0 0 0
- added joint base_link_base_gps_joint: type fixed, parent base_link, child base_gps, origin xyz=0 0 0 rpy=0 0 0
- added joint base_link_base_gyro_joint: type fixed, parent base_link, child base_gyro, origin xyz=0 0 0 rpy=0 0 0
- added joint base_link_base_inertial_joint: type fixed, parent base_link, child base_inertial, origin xyz=0 0 0 rpy=0 0 0
- added joint base_link_base_link_inertia_joint: type fixed, parent base_link, child base_link_inertia, origin xyz=0 0 0.1545 rpy=0 0 0
- added joint hingejoint: type fixed, parent base_link, child cw_hr_link, origin xyz=-0.25 -0.185 0.005 rpy=0 0 0, axis 0 1 0
- added joint hingejoint_0: type fixed, parent base_link, child cw_hl_link, origin xyz=-0.25 0.185 0.005 rpy=0 0 0, axis 0 1 0
- added joint hingejoint_1: type fixed, parent base_link, child cw_fr_link, origin xyz=0.25 -0.185 0.005 rpy=0 0 0, axis 0 1 0
- added joint hingejoint_2: type fixed, parent base_link, child cw_fl_link, origin xyz=0.25 0.185 0.005 rpy=0 0 0, axis 0 1 0
- added joint joint1: type revolute, parent arm_base, child link1, origin xyz=0 0 0.155 rpy=0 0 3.141592, axis 0 0 1, limit lower=-2.7925 upper=2.7925 effort=123 velocity=2.0944
- added joint joint2: type revolute, parent link1, child link2, origin xyz=0 0.03 0.21 rpy=0 0.785398 0, axis 0 1 0, limit lower=-2.2689 upper=2.2689 effort=123 velocity=2.0944
- added joint joint3: type revolute, parent link2, child link3, origin xyz=0 0.035 0.205 rpy=0 0 0, axis 0 0 1, limit lower=-2.9671 upper=2.9671 effort=64 velocity=2.4435
- added joint joint4: type revolute, parent link3, child link4, origin xyz=-0.02 -0.03 0.19 rpy=-3.141591 1.396263 0.000002, axis 0 1 0, limit lower=-1.8675 upper=2.6878 effort=64 velocity=2.4435
- added joint joint5: type revolute, parent link4, child link5, origin xyz=-0.02 0.025 0.195 rpy=0 0 3.141592, axis 0 0 1, limit lower=-2.9671 upper=2.9671 effort=39 velocity=4.8869
- added joint joint6: type revolute, parent link5, child link6, origin xyz=0 0.03 0.19 rpy=0 0 0, axis 0 1 0, limit lower=-1.3963 upper=4.5379 effort=39 velocity=4.8869
- added joint joint7: type revolute, parent link6, child link7, origin xyz=-0.055 0.07 0.11 rpy=0 -1.570796 0, axis 0 0 1, limit lower=-2.9671 upper=2.9671 effort=39 velocity=4.8869

Commit message: correct urdf

File: urdf2model/models/mabimobile/mabi_mobile.urdf (robot description, URDF)
Before this commit: robot mabi_mobile, 20 links, 19 joints
Links:
- added link flange
- link arm_base: mass None -> 3.7; geometry collision mesh filename=meshes/rizon4s/collision/link0.stl; visual mesh filename=meshes/rizon4s/visual/link0.obj
- link link1: mass None -> 3.7; geometry collision mesh filename=meshes/rizon4s/collision/link1.stl; visual mesh filename=meshes/rizon4s/visual/link1.obj
- link link2: mass None -> 2.7; geometry collision mesh filename=meshes/rizon4s/collision/link2.stl; visual mesh filename=meshes/rizon4s/visual/link2.obj
- link link3: mass None -> 2.4; geometry collision mesh filename=meshes/rizon4s/collision/link3.stl; visual mesh filename=meshes/rizon4s/visual/link3.obj
- link link4: mass None -> 2.4; geometry collision mesh filename=meshes/rizon4s/collision/link4.stl; visual mesh filename=meshes/rizon4s/visual/link4.obj
- link link5: mass None -> 2.4; geometry collision mesh filename=meshes/rizon4s/collision/link5.stl; visual mesh filename=meshes/rizon4s/visual/link5.obj
- link link6: mass None -> 2.1; geometry collision mesh filename=meshes/rizon4s/collision/link6.stl; visual mesh filename=meshes/rizon4s/visual/link6.obj
- link link7: mass None -> 1.4; geometry collision mesh filename=meshes/rizon4s/collision/link7.stl; visual mesh filename=meshes/rizon4s/visual/link7.obj
Joints:
- added joint link7_to_flange: type fixed, parent link7, child flange, origin xyz=0.0 0.0 0.124 rpy=0.0 0.0 -3.141592653589793
- joint joint1: origin xyz=0 0 0.155 rpy=0 0 3.141592 -> xyz=0.0 0.0 0.155 rpy=0.0 0.0 -3.141592653589793
- joint joint2: origin xyz=0 0.03 0.21 rpy=0 0.785398 0 -> xyz=0.0 0.03 0.21 rpy=0.0 0.0 0.0
- joint joint3: origin xyz=0 0.035 0.205 rpy=0 0 0 -> xyz=0.0 0.035 0.205 rpy=0.0 0.0 0.0
- joint joint4: origin xyz=-0.02 -0.03 0.19 rpy=-3.141591 1.396263 0.000002 -> xyz=-0.02 -0.03 0.19 rpy=0.0 0.0 -3.141592653589793
- joint joint5: origin xyz=-0.02 0.025 0.195 rpy=0 0 3.141592 -> xyz=-0.02 0.025 0.195 rpy=0.0 0.0 -3.141592653589793
- joint joint6: origin xyz=0 0.03 0.19 rpy=0 0 0 -> xyz=0.0 0.03 0.19 rpy=0.0 0.0 0.0
- joint joint7: origin xyz=-0.055 0.07 0.11 rpy=0 -1.570796 0 -> xyz=-0.055 0.07 0.11 rpy=0.0 -1.5707963478683205 0.0

Commit message: use real base model

File: urdf2model/models/mabimobile/mabi_mobile.urdf (robot description, URDF)
Before this commit: robot mabi_mobile, 21 links, 20 joints
Links:
- removed link L_WHEEL
- removed link R_WHEEL
- removed link base_acc
- removed link base_gps
- removed link base_gyro
- removed link base_inertial
- removed link base_link_inertia
- removed link cw_fl_link
- removed link cw_fr_link
- removed link cw_hl_link
- removed link cw_hr_link
- added link fl_wheel, mass 0.42252; collision cylinder length=0.08 radius=0.075; visual mesh filename=meshes/wheel.stl
- added link fr_wheel, mass 0.42252; collision cylinder length=0.08 radius=0.075; visual mesh filename=meshes/wheel.stl
- added link rl_wheel, mass 0.42252; collision cylinder length=0.08 radius=0.075; visual mesh filename=meshes/wheel.stl
- added link rr_wheel, mass 0.42252; collision cylinder length=0.08 radius=0.075; visual mesh filename=meshes/wheel.stl
- link base_link: mass None -> 19.7081876920141; geometry collision box size=1.020 0.585 0.6785; visual mesh filename=meshes/base.stl
- link link7: mass 1.4 -> 2.27
Joints:
- removed joint L_WHEEL
- removed joint R_WHEEL
- removed joint base_link_base_acc_joint
- removed joint base_link_base_gps_joint
- removed joint base_link_base_gyro_joint
- removed joint base_link_base_inertial_joint
- removed joint base_link_base_link_inertia_joint
- removed joint hingejoint
- removed joint hingejoint_0
- removed joint hingejoint_1
- removed joint hingejoint_2
- added joint fl_wheel_joint: type fixed, parent base_link, child fl_wheel, origin xyz=0.305 0.3 0 rpy=0 0 0, axis 0 1 0
- added joint fr_wheel_joint: type fixed, parent base_link, child fr_wheel, origin xyz=0.305 -0.3 0 rpy=0 0 0, axis 0 1 0
- added joint rl_wheel_joint: type fixed, parent base_link, child rl_wheel, origin xyz=-0.305 0.3 0 rpy=0 0 0, axis 0 1 0
- added joint rr_wheel_joint: type fixed, parent base_link, child rr_wheel, origin xyz=-0.305 -0.3 0 rpy=0 0 0, axis 0 1 0
- joint base_link_arm_base_joint: origin xyz=0 0 0.309 rpy=0 0 0 -> xyz=0.3 0 0.69 rpy=0 0 0

Commit message: add gripper length in model

File: urdf2model/models/mabimobile/mabi_mobile.urdf (robot description, URDF)
Before this commit: robot mabi_mobile, 14 links, 13 joints
Joints:
- joint link7_to_flange: origin xyz=0.0 0.0 0.124 rpy=0.0 0.0 -3.141592653589793 -> xyz=0.0 0.0 0.334 rpy=0.0 0.0 -3.141592653589793
